File: i2c_transceiver.kicad_sch (KiCad schematic)
At the start: 11 parts, among them U2 PCA9306DP

Commit message: Updates 2
Connections:
- net +3V3 is gone; now on net +3.3V: +3.3V2.1, U2.2 (VREF1)
Changed lines of the file:
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@@
   (junction (at 125.73 90.17) (diameter 0) (color 0 0 0 0)
   )
+  (junction (at 146.05 77.47) (diameter 0) (color 0 0 0 0)
+  )
   (junction (at 180.34 90.17) (diameter 0) (color 0 0 0 0)
   )
-  (junction (at 146.05 77.47) (diameter 0) (color 0 0 0 0)
-  )
   (junction (at 165.1 90.17) (diameter 0) (color 0 0 0 0)
   )
@@
   )
   (wire (pts (xy 158.75 92.71) (xy 171.45 92.71))
+    (stroke (width 0) (type default))
+  )
+  (wire (pts (xy 146.05 74.93) (xy 146.05 77.47))
     (stroke (width 0) (type default))
   )
@@
   )
   (symbol (lib_id "Connector:TestPoint") (at 140.97 71.12 0) (unit 1)
-    (in_bom yes) (on_board yes) (dnp no) (fields_autoplaced)
+    (in_bom yes) (on_board yes) (dnp no)
     (property "Reference" "+3.3V2" (at 143.51 66.548 0)
       (effects (font (size 1.27 1.27)) (justify left))
     )
-    (property "Value" "TP3.3v" (at 143.51 69.088 0)
+    (property "Value" "TP3.3v" (at 144.78 64.77 0)
       (effects (font (size 1.27 1.27)) (justify left))
     )
@@
     )
   )
-  (symbol (lib_id "power:+3V3") (at 146.05 77.47 0) (unit 1)
-    (in_bom yes) (on_board yes) (dnp no)
-    (property "Reference" "#PWR028" (at 146.05 81.28 0)
-      (effects (font (size 1.27 1.27)) hide)
-    )
-    (property "Value" "+3V3" (at 146.431 73.0758 0)
-      (effects (font (size 1.27 1.27)))
-    )
-    (property "Footprint" "" (at 146.05 77.47 0)
-      (effects (font (size 1.27 1.27)) hide)
-    )
-    (property "Datasheet" "" (at 146.05 77.47 0)
-      (effects (font (size 1.27 1.27)) hide)
-    )
-    (pin "1")
-    (instances
-      (project "LTP305_ESP32_CLOCK"
-        (path "/c007e288-8439-49d9-bbdf-49724c34958c"
-          (reference "#PWR028") (unit 1)
-        )
-      )
-      (project "ltp_kikad"
+  (symbol (lib_id "power:+3.3V") (at 146.05 74.93 0) (unit 1)
+    (in_bom yes) (on_board yes) (dnp no) (fields_autoplaced)
+    (property "Reference" "#PWR058" (at 146.05 78.74 0)
+      (effects (font (size 1.27 1.27)) hide)
+    )
+    (property "Value" "+3.3V" (at 146.05 69.85 0)
+      (effects (font (size 1.27 1.27)))
+    )
+    (property "Footprint" "" (at 146.05 74.93 0)
+      (effects (font (size 1.27 1.27)) hide)
+    )
+    (property "Datasheet" "" (at 146.05 74.93 0)
+      (effects (font (size 1.27 1.27)) hide)
+    )
+    (pin "1")
+    (instances
+      (project "ltp_kikad"
+        (path "/eed35b77-cbf9-4596-9b17-2558f81058ba"
+          (reference "#PWR058") (unit 1)
+        )
         (path "/eed35b77-cbf9-4596-9b17-2558f81058ba/2fb8f433-d537-4253-8cc8-f6d42368ed9e"
           (reference "#PWR070") (unit 1)
