File: _autosave-ltp_kikad.kicad_sch (KiCad schematic)
At the start: 7 parts, among them J2 RPi_GPIO

Commit message: Add inductor
Other:
- added sheet dc_dc (dc.kicad_sch)
Changed lines of the file:
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@@
+    )
+  )
+  (sheet (at 115.57 33.02) (size 59.69 10.16) (fields_autoplaced)
+    (stroke (width 0.1524) (type solid))
+    (fill (color 0 0 0 0.0000))
+    (property "Sheetname" "dc_dc" (at 115.57 32.3084 0)
+      (effects (font (size 1.27 1.27)) (justify left bottom))
+    )
+    (property "Sheetfile" "dc.kicad_sch" (at 115.57 43.7646 0)
+      (effects (font (size 1.27 1.27)) (justify left top))
+    )
+    (property "Field2" "" (at 115.57 33.02 0)
+      (effects (font (size 1.27 1.27)) hide)
+    )
+    (instances
+      (project "ltp_kikad"
+        (path "/eed35b77-cbf9-4596-9b17-2558f81058ba" (page "5"))
+      )
     )
   )
