File: dcdc.kicad_sch (KiCad schematic)
At the start: 5 parts, among them IC3 ME2108A33PG

Commit message: Add title block
Other:
- company: (none) -> Andrew Tudoroi
- title: (none) -> Pitanga HAT
Changed lines of the file:
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@@
 (kicad_sch (version 20230121) (generator eeschema)
   (paper "A4")
+  (title_block
+    (title "Pitanga HAT")
+    (date "2023-10-20")
+    (rev "2.1")
+    (company "Andrew Tudoroi")
+  )
   (junction (at 167.64 77.47) (diameter 0) (color 0 0 0 0)
   )
