File: dcdc.kicad_sch (KiCad schematic)
At the start: 5 parts, among them IC3 ME2108A33PG

Commit message: Fix decimal point connection on ds4, add info to title block
Other:
- company: (none) -> Andrew Tudoroi
- title: (none) -> Pitanga HAT
Changed lines of the file:
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@@
 (kicad_sch (version 20230121) (generator eeschema)
   (paper "A4")
+  (title_block
+    (title "Pitanga HAT")
+    (date "2023-10-19")
+    (rev "2.1")
+    (company "Andrew Tudoroi")
+  )
   (junction (at 167.64 77.47) (diameter 0) (color 0 0 0 0)
   )

Commit message: Piatnag_5_bt
Parts:
- removed C7 (x2): 15uF, Capacitor_SMD:C_1210_3225Metric_Pad1.33x2.70mm_HandSolder, symbol Device:C_Small
- removed D5: SS14, Library:DIOM5127X261N, symbol SS14:SS14
- removed IC3: ME2108A33PG, Package_TO_SOT_SMD:SOT-89-3_Handsoldering, symbol ME2108A33M3G:ME2108A33PG
- removed L1: 220uH, Library:WE-SPC_48XX78, symbol Device:L
