File: i2c_connector.kicad_sch (KiCad schematic)
At the start: 11 parts, among them J3 SM04B-SRSS-TB(LF)(SN)

Commit message: Finilize small buttons
Other:
- moved on the sheet: C7
Changed lines of the file:
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@@
     (stroke (width 0) (type default))
   )
-  (wire (pts (xy 58.42 71.12) (xy 58.42 76.2))
-    (stroke (width 0) (type default))
-  )
-  (wire (pts (xy 85.09 71.12) (xy 85.09 76.2))
+  (wire (pts (xy 62.23 71.12) (xy 62.23 76.2))
+    (stroke (width 0) (type default))
+  )
+  (wire (pts (xy 80.01 71.12) (xy 80.01 76.2))
     (stroke (width 0) (type default))
   )
@@
     (stroke (width 0) (type solid))
   )
-  (wire (pts (xy 58.42 81.28) (xy 58.42 86.36))
-    (stroke (width 0) (type default))
-  )
-  (wire (pts (xy 71.12 71.12) (xy 85.09 71.12))
+  (wire (pts (xy 62.23 81.28) (xy 62.23 86.36))
     (stroke (width 0) (type default))
   )
@@
     (stroke (width 0) (type solid))
   )
+  (wire (pts (xy 71.12 71.12) (xy 80.01 71.12))
+    (stroke (width 0) (type default))
+  )
   (wire (pts (xy 154.94 143.51) (xy 172.72 143.51))
     (stroke (width 0) (type default))
@@
     (stroke (width 0) (type solid))
   )
-  (wire (pts (xy 85.09 81.28) (xy 85.09 86.36))
+  (wire (pts (xy 80.01 81.28) (xy 80.01 86.36))
     (stroke (width 0) (type default))
   )
@@
     (stroke (width 0) (type solid))
   )
-  (wire (pts (xy 58.42 71.12) (xy 71.12 71.12))
+  (wire (pts (xy 62.23 71.12) (xy 71.12 71.12))
     (stroke (width 0) (type default))
   )
@@
     )
   )
-  (symbol (lib_id "Device:C_Small") (at 85.09 78.74 180) (unit 1)
-    (in_bom yes) (on_board yes) (dnp no)
-    (property "Reference" "C7" (at 90.17 77.47 0)
-      (effects (font (size 1.27 1.27)))
-    )
-    (property "Value" "15uF" (at 90.17 80.01 0)
-      (effects (font (size 1.27 1.27)))
-    )
-    (property "Footprint" "Capacitor_SMD:C_1210_3225Metric_Pad1.33x2.70mm_HandSolder" (at 85.09 78.74 0)
-      (effects (font (size 1.27 1.27)) hide)
-    )
-    (property "Datasheet" "~" (at 85.09 78.74 0)
+  (symbol (lib_id "Device:C_Small") (at 80.01 78.74 180) (unit 1)
+    (in_bom yes) (on_board yes) (dnp no)
+    (property "Reference" "C7" (at 85.09 77.47 0)
+      (effects (font (size 1.27 1.27)))
+    )
+    (property "Value" "15uF" (at 85.09 80.01 0)
+      (effects (font (size 1.27 1.27)))
+    )
+    (property "Footprint" "Capacitor_SMD:C_1210_3225Metric_Pad1.33x2.70mm_HandSolder" (at 80.01 78.74 0)
+      (effects (font (size 1.27 1.27)) hide)
+    )
+    (property "Datasheet" "~" (at 80.01 78.74 0)
       (effects (font (size 1.27 1.27)) hide)
     )
@@
     )
   )
-  (symbol (lib_id "Device:C_Small") (at 58.42 78.74 180) (unit 1)
-    (in_bom yes) (on_board yes) (dnp no)
-    (property "Reference" "C7" (at 63.5 77.47 0)
-      (effects (font (size 1.27 1.27)))
-    )
-    (property "Value" "15uF" (at 63.5 80.01 0)
-      (effects (font (size 1.27 1.27)))
-    )
-    (property "Footprint" "Capacitor_SMD:C_1210_3225Metric_Pad1.33x2.70mm_HandSolder" (at 58.42 78.74 0)
-      (effects (font (size 1.27 1.27)) hide)
-    )
-    (property "Datasheet" "~" (at 58.42 78.74 0)
+  (symbol (lib_id "Device:C_Small") (at 62.23 78.74 180) (unit 1)
+    (in_bom yes) (on_board yes) (dnp no)
+    (property "Reference" "C7" (at 67.31 77.47 0)
+      (effects (font (size 1.27 1.27)))
+    )
+    (property "Value" "15uF" (at 67.31 80.01 0)
+      (effects (font (size 1.27 1.27)))
+    )
+    (property "Footprint" "Capacitor_SMD:C_1210_3225Metric_Pad1.33x2.70mm_HandSolder" (at 62.23 78.74 0)
+      (effects (font (size 1.27 1.27)) hide)
+    )
+    (property "Datasheet" "~" (at 62.23 78.74 0)
       (effects (font (size 1.27 1.27)) hide)
     )
@@
     )
   )
-  (symbol (lib_id "power:GND") (at 85.09 86.36 0) (unit 1)
-    (in_bom yes) (on_board yes) (dnp no)
-    (property "Reference" "#PWR033" (at 85.09 92.71 0)
-      (effects (font (size 1.27 1.27)) hide)
-    )
-    (property "Value" "GND" (at 85.217 90.7542 0)
-      (effects (font (size 1.27 1.27)))
-    )
-    (property "Footprint" "" (at 85.09 86.36 0)
-      (effects (font (size 1.27 1.27)) hide)
-    )
-    (property "Datasheet" "" (at 85.09 86.36 0)
+  (symbol (lib_id "power:GND") (at 80.01 86.36 0) (unit 1)
+    (in_bom yes) (on_board yes) (dnp no)
+    (property "Reference" "#PWR033" (at 80.01 92.71 0)
+      (effects (font (size 1.27 1.27)) hide)
+    )
+    (property "Value" "GND" (at 80.137 90.7542 0)
+      (effects (font (size 1.27 1.27)))
+    )
+    (property "Footprint" "" (at 80.01 86.36 0)
+      (effects (font (size 1.27 1.27)) hide)
+    )
+    (property "Datasheet" "" (at 80.01 86.36 0)
       (effects (font (size 1.27 1.27)) hide)
     )
@@
     )
   )
-  (symbol (lib_id "power:GND") (at 58.42 86.36 0) (unit 1)
-    (in_bom yes) (on_board yes) (dnp no)
-    (property "Reference" "#PWR033" (at 58.42 92.71 0)
-      (effects (font (size 1.27 1.27)) hide)
-    )
-    (property "Value" "GND" (at 58.547 90.7542 0)
-      (effects (font (size 1.27 1.27)))
-    )
-    (property "Footprint" "" (at 58.42 86.36 0)
-      (effects (font (size 1.27 1.27)) hide)
-    )
-    (property "Datasheet" "" (at 58.42 86.36 0)
-      (effects (font (size 1.27 1.27)) hide)
-    )
+  (symbol (lib_id "power:GND") (at 62.23 86.36 0) (unit 1)
+    (in_bom yes) (on_board yes) (dnp no)
+    (property "Reference" "#PWR033" (at 62.23 92.71 0)
+      (effects (font (size 1.27 1.27)) hide)
+    )
+    (property "Value" "GND" (at 62.357 90.7542 0)
+      (effects (font (size 1.27 1.27)))
+    )
+    (property "Footprint" "" (at 62.23 86.36 0)
+      (effects (font (size 1.27 1.27)) hide)
+    )
+    (property "Datasheet" "" (at 62.23 86.36 0)
+      (effects (font (size 1.27 1.27)) hide)
+    )
