File: i2c_connector.kicad_sch (KiCad schematic)
At the start: 11 parts, among them J3 SM04B-SRSS-TB(LF)(SN)

Commit message: Move from 4 layer to 2, complete roting, separate 5v for led driver and 3v i2c power
Parts:
- removed C11 (x2): 10uF, Capacitor_SMD:C_0603_1608Metric, symbol Device:C_Small
- removed J3: SM04B-SRSS-TB(LF)(SN), ltp_kikad:JST_SM04B-SRSS-TB(LF)(SN), symbol SM04B-SRSS-TB_LF__SN_:SM04B-SRSS-TB(LF)(SN)
- removed R3: 10k, Resistor_SMD:R_0603_1608Metric, symbol Device:R
- removed R3: 47k, Resistor_SMD:R_0603_1608Metric, symbol Device:R
- added C11: 10uF, Capacitor_SMD:C_0603_1608Metric, symbol Device:C_Small
Connections:
- net +3V3: now also C11.1
- net GND: now also C11.2
