File: i2c_tramsciever.kicad_sch (KiCad schematic)
At the start: 6 parts, among them U2 PCA9306DP

Commit message: Add title block
Other:
- company: (none) -> Andrew Tudoroi
- title: (none) -> Pitanga HAT
Changed lines of the file:
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@@
 (kicad_sch (version 20230121) (generator eeschema)
   (paper "A4")
+  (title_block
+    (title "Pitanga HAT")
+    (date "2023-10-20")
+    (rev "2.1")
+    (company "Andrew Tudoroi")
+  )
   (junction (at 146.05 72.39) (diameter 0) (color 0 0 0 0)
   )

Commit message: Finilize small buttons
Parts:
- added JP1, JP2: SolderJumper_2_Open, Jumper:SolderJumper-2_P1.3mm_Open_RoundedPad1.0x1.5mm, symbol Jumper:SolderJumper_2_Open
Connections:
- net 5vSCL: now also JP1.2 (B)
- net 5vSDA: now also JP2.2 (B)
- net SCL: now also JP1.1 (A)
- net SDA: now also JP2.1 (A)
Changed lines of the file:
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@@
   (junction (at 152.4 85.09) (diameter 0) (color 0 0 0 0)
   )
+  (junction (at 113.03 87.63) (diameter 0) (color 0 0 0 0)
+  )
+  (junction (at 118.11 85.09) (diameter 0) (color 0 0 0 0)
+  )
   (junction (at 133.35 69.85) (diameter 0) (color 0 0 0 0)
   )
@@
     (stroke (width 0) (type default))
   )
+  (wire (pts (xy 132.08 123.19) (xy 113.03 123.19))
+    (stroke (width 0) (type default))
+  )
   (wire (pts (xy 133.35 67.31) (xy 133.35 69.85))
     (stroke (width 0) (type default))
   )
+  (wire (pts (xy 118.11 85.09) (xy 125.73 85.09))
+    (stroke (width 0) (type default))
+  )
   (wire (pts (xy 152.4 59.69) (xy 146.05 59.69))
     (stroke (width 0) (type default))
@@
     (stroke (width 0) (type default))
   )
+  (wire (pts (xy 113.03 123.19) (xy 113.03 87.63))
+    (stroke (width 0) (type default))
+  )
   (wire (pts (xy 152.4 85.09) (xy 168.91 85.09))
     (stroke (width 0) (type default))
   )
-  (wire (pts (xy 107.95 85.09) (xy 125.73 85.09))
+  (wire (pts (xy 139.7 123.19) (xy 158.75 123.19))
+    (stroke (width 0) (type default))
+  )
+  (wire (pts (xy 107.95 85.09) (xy 118.11 85.09))
     (stroke (width 0) (type default))
   )
@@
     (stroke (width 0) (type default))
   )
+  (wire (pts (xy 118.11 113.03) (xy 118.11 85.09))
+    (stroke (width 0) (type default))
+  )
   (wire (pts (xy 146.05 59.69) (xy 146.05 62.23))
     (stroke (width 0) (type default))
   )
+  (wire (pts (xy 152.4 113.03) (xy 152.4 85.09))
+    (stroke (width 0) (type default))
+  )
   (wire (pts (xy 171.45 59.69) (xy 158.75 59.69))
     (stroke (width 0) (type default))
@@
     (stroke (width 0) (type default))
   )
-  (wire (pts (xy 107.95 87.63) (xy 125.73 87.63))
+  (wire (pts (xy 107.95 87.63) (xy 113.03 87.63))
+    (stroke (width 0) (type default))
+  )
+  (wire (pts (xy 158.75 123.19) (xy 158.75 87.63))
+    (stroke (width 0) (type default))
+  )
+  (wire (pts (xy 132.08 113.03) (xy 118.11 113.03))
     (stroke (width 0) (type default))
   )
@@
   )
   (wire (pts (xy 133.35 69.85) (xy 133.35 72.39))
+    (stroke (width 0) (type default))
+  )
+  (wire (pts (xy 113.03 87.63) (xy 125.73 87.63))
+    (stroke (width 0) (type default))
+  )
+  (wire (pts (xy 139.7 113.03) (xy 152.4 113.03))
     (stroke (width 0) (type default))
   )
@@
     )
   )
+  (symbol (lib_id "Jumper:SolderJumper_2_Open") (at 135.89 113.03 0) (unit 1)
+    (in_bom yes) (on_board yes) (dnp no) (fields_autoplaced)
+    (property "Reference" "JP1" (at 135.89 106.68 0)
+      (effects (font (size 1.27 1.27)))
+    )
+    (property "Value" "SolderJumper_2_Open" (at 135.89 109.22 0)
+      (effects (font (size 1.27 1.27)))
+    )
+    (property "Footprint" "Jumper:SolderJumper-2_P1.3mm_Open_RoundedPad1.0x1.5mm" (at 135.89 113.03 0)
+      (effects (font (size 1.27 1.27)) hide)
+    )
+    (property "Datasheet" "~" (at 135.89 113.03 0)
+      (effects (font (size 1.27 1.27)) hide)
+    )
+    (pin "1")
+    (pin "2")
+    (instances
+      (project "ltp_kikad"
+        (path "/eed35b77-cbf9-4596-9b17-2558f81058ba/e885c20e-c513-4e27-ac27-692e5f196b61"
+          (reference "JP1") (unit 1)
+        )
+      )
+    )
+  )
   (symbol (lib_id "power:GND") (at 171.45 71.12 0) (unit 1)
     (in_bom yes) (on_board yes) (dnp no)
@@
         )
       )
+    )
+  )
+  (symbol (lib_id "Jumper:SolderJumper_2_Open") (at 135.89 123.19 0) (unit 1)
+    (in_bom yes) (on_board yes) (dnp no) (fields_autoplaced)
+    (property "Reference" "JP2" (at 135.89 116.84 0)
+      (effects (font (size 1.27 1.27)))
+    )
+    (property "Value" "SolderJumper_2_Open" (at 135.89 119.38 0)
+      (effects (font (size 1.27 1.27)))
+    )
+    (property "Footprint" "Jumper:SolderJumper-2_P1.3mm_Open_RoundedPad1.0x1.5mm" (at 135.89 123.19 0)
+      (effects (font (size 1.27 1.27)) hide)
+    )
+    (property "Datasheet" "~" (at 135.89 123.19 0)
+      (effects (font (size 1.27 1.27)) hide)
+    )
+    (pin "1")
+    (pin "2")
+    (instances
+      (project "ltp_kikad"
+        (path "/eed35b77-cbf9-4596-9b17-2558f81058ba/e885c20e-c513-4e27-ac27-692e5f196b61"
+          (reference "JP2") (unit 1)
+        )
+      )
