File: stm32_mcu.kicad_sch (KiCad schematic)
At the start: 9 parts, among them J4 Conn_ARM_SWD_TagConnect_TC203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, J5 Conn_01x08_Pin, J6 Conn_01x08_Pin, U1 STM32G031J6Mx

Commit message: Add title block
Other:
- company: (none) -> Andrew Tudoroi
- title: (none) -> Pitanga HAT
Changed lines of the file:
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@@
 (kicad_sch (version 20230121) (generator eeschema)
   (paper "A4")
+  (title_block
+    (title "Pitanga HAT")
+    (date "2023-10-20")
+    (rev "2.1")
+    (company "Andrew Tudoroi")
+  )
   (junction (at 149.86 118.11) (diameter 0) (color 0 0 0 0)
   )

Commit message: Finilize small buttons
Other:
- moved on the sheet: C11
Changed lines of the file:
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@@
   (junction (at 198.12 80.01) (diameter 0) (color 0 0 0 0)
   )
+  (junction (at 87.63 53.34) (diameter 0) (color 0 0 0 0)
+  )
   (junction (at 196.85 77.47) (diameter 0) (color 0 0 0 0)
   )
@@
   (junction (at 184.15 82.55) (diameter 0) (color 0 0 0 0)
   )
-  (junction (at 115.57 57.15) (diameter 0) (color 0 0 0 0)
-  )
   (wire (pts (xy 123.19 82.55) (xy 125.73 82.55))
     (stroke (width 0) (type default))
@@
     (stroke (width 0) (type default))
   )
-  (wire (pts (xy 119.38 57.15) (xy 119.38 63.5))
+  (wire (pts (xy 95.25 53.34) (xy 95.25 59.69))
     (stroke (width 0) (type default))
   )
@@
     (stroke (width 0) (type default))
   )
-  (wire (pts (xy 133.35 124.46) (xy 133.35 130.81))
+  (wire (pts (xy 78.74 53.34) (xy 78.74 59.69))
     (stroke (width 0) (type default))
   )
@@
     (stroke (width 0) (type default))
   )
-  (wire (pts (xy 111.76 57.15) (xy 111.76 63.5))
+  (wire (pts (xy 87.63 53.34) (xy 87.63 59.69))
     (stroke (width 0) (type default))
   )
@@
     (stroke (width 0) (type default))
   )
-  (wire (pts (xy 111.76 57.15) (xy 115.57 57.15))
+  (wire (pts (xy 87.63 53.34) (xy 95.25 53.34))
     (stroke (width 0) (type default))
   )
@@
     (stroke (width 0) (type default))
   )
+  (wire (pts (xy 78.74 53.34) (xy 87.63 53.34))
+    (stroke (width 0) (type default))
+  )
   (wire (pts (xy 257.81 91.44) (xy 257.81 92.71))
     (stroke (width 0) (type default))
   )
-  (wire (pts (xy 115.57 54.61) (xy 115.57 57.15))
-    (stroke (width 0) (type default))
-  )
-  (wire (pts (xy 119.38 57.15) (xy 115.57 57.15))
+  (wire (pts (xy 87.63 50.8) (xy 87.63 53.34))
     (stroke (width 0) (type default))
   )
@@
     )
   )
-  (symbol (lib_id "power:GND") (at 119.38 68.58 0) (unit 1)
-    (in_bom yes) (on_board yes) (dnp no)
-    (property "Reference" "#PWR038" (at 119.38 74.93 0)
-      (effects (font (size 1.27 1.27)) hide)
-    )
-    (property "Value" "GND" (at 119.507 72.9742 0)
-      (effects (font (size 1.27 1.27)))
-    )
-    (property "Footprint" "" (at 119.38 68.58 0)
-      (effects (font (size 1.27 1.27)) hide)
-    )
-    (property "Datasheet" "" (at 119.38 68.58 0)
+  (symbol (lib_id "power:GND") (at 95.25 64.77 0) (unit 1)
+    (in_bom yes) (on_board yes) (dnp no)
+    (property "Reference" "#PWR038" (at 95.25 71.12 0)
+      (effects (font (size 1.27 1.27)) hide)
+    )
+    (property "Value" "GND" (at 95.377 69.1642 0)
+      (effects (font (size 1.27 1.27)))
+    )
+    (property "Footprint" "" (at 95.25 64.77 0)
+      (effects (font (size 1.27 1.27)) hide)
+    )
+    (property "Datasheet" "" (at 95.25 64.77 0)
       (effects (font (size 1.27 1.27)) hide)
     )
@@
         (path "/eed35b77-cbf9-4596-9b17-2558f81058ba/c7f9496d-fb5e-4ce7-92b5-54c2d3a6681a"
           (reference "#PWR028") (unit 1)
-        )
-      )
-    )
-  )
-  (symbol (lib_id "rpi-pico-debugger-shoe-rescue:+3.3V-power") (at 133.35 124.46 0) (unit 1)
-    (in_bom yes) (on_board yes) (dnp no)
-    (property "Reference" "#PWR0104" (at 133.35 128.27 0)
-      (effects (font (size 1.27 1.27)) hide)
-    )
-    (property "Value" "+3.3V" (at 133.731 120.0658 0)
-      (effects (font (size 1.27 1.27)))
-    )
-    (property "Footprint" "" (at 133.35 124.46 0)
-      (effects (font (size 1.27 1.27)) hide)
-    )
-    (property "Datasheet" "" (at 133.35 124.46 0)
-      (effects (font (size 1.27 1.27)) hide)
-    )
-    (pin "1")
-    (instances
-      (project "rpi-pico-debugger-shoe"
-        (path "/aad74d97-f116-4a83-b498-c8cb2f4b4e35"
-          (reference "#PWR0104") (unit 1)
-        )
-      )
-      (project "ltp_kikad"
-        (path "/eed35b77-cbf9-4596-9b17-2558f81058ba"
-          (reference "#PWR0119") (unit 1)
-        )
-        (path "/eed35b77-cbf9-4596-9b17-2558f81058ba/c7f9496d-fb5e-4ce7-92b5-54c2d3a6681a"
-          (reference "#PWR030") (unit 1)
         )
       )
@@
     )
   )
-  (symbol (lib_id "power:GND") (at 111.76 68.58 0) (unit 1)
-    (in_bom yes) (on_board yes) (dnp no)
-    (property "Reference" "#PWR038" (at 111.76 74.93 0)
-      (effects (font (size 1.27 1.27)) hide)
-    )
-    (property "Value" "GND" (at 111.887 72.9742 0)
-      (effects (font (size 1.27 1.27)))
-    )
-    (property "Footprint" "" (at 111.76 68.58 0)
-      (effects (font (size 1.27 1.27)) hide)
-    )
-    (property "Datasheet" "" (at 111.76 68.58 0)
+  (symbol (lib_id "power:GND") (at 87.63 64.77 0) (unit 1)
+    (in_bom yes) (on_board yes) (dnp no)
+    (property "Reference" "#PWR038" (at 87.63 71.12 0)
+      (effects (font (size 1.27 1.27)) hide)
+    )
+    (property "Value" "GND" (at 87.757 69.1642 0)
+      (effects (font (size 1.27 1.27)))
+    )
+    (property "Footprint" "" (at 87.63 64.77 0)
+      (effects (font (size 1.27 1.27)) hide)
+    )
+    (property "Datasheet" "" (at 87.63 64.77 0)
       (effects (font (size 1.27 1.27)) hide)
     )
@@
     )
   )
-  (symbol (lib_id "Device:C_Small") (at 133.35 133.35 0) (unit 1)
-    (in_bom yes) (on_board yes) (dnp no)
-    (property "Reference" "C11" (at 135.6868 132.1816 0)
+  (symbol (lib_id "Device:C_Small") (at 78.74 62.23 0) (unit 1)
+    (in_bom yes) (on_board yes) (dnp no)
+    (property "Reference" "C11" (at 81.0768 61.0616 0)
       (effects (font (size 1.27 1.27)) (justify left))
     )
-    (property "Value" "0.1uF" (at 128.27 135.89 0)
+    (property "Value" "0.1uF" (at 73.66 64.77 0)
       (effects (font (size 1.27 1.27)) (justify left))
     )
-    (property "Footprint" "Capacitor_SMD:C_0402_1005Metric" (at 133.35 133.35 0)
-      (effects (font (size 1.27 1.27)) hide)
-    )
-    (property "Datasheet" "~" (at 133.35 133.35 0)
+    (property "Footprint" "Capacitor_SMD:C_0402_1005Metric" (at 78.74 62.23 0)
+      (effects (font (size 1.27 1.27)) hide)
+    )
+    (property "Datasheet" "~" (at 78.74 62.23 0)
       (effects (font (size 1.27 1.27)) hide)
     )
@@
     )
   )
-  (symbol (lib_id "rpi-pico-debugger-shoe-rescue:+3.3V-power") (at 115.57 54.61 0) (unit 1)
-    (in_bom yes) (on_board yes) (dnp no)
-    (property "Reference" "#PWR0104" (at 115.57 58.42 0)
-      (effects (font (size 1.27 1.27)) hide)
-    )
-    (property "Value" "+3.3V" (at 115.951 50.2158 0)
-      (effects (font (size 1.27 1.27)))
-    )
-    (property "Footprint" "" (at 115.57 54.61 0)
-      (effects (font (size 1.27 1.27)) hide)
-    )
-    (property "Datasheet" "" (at 115.57 54.61 0)
+  (symbol (lib_id "rpi-pico-debugger-shoe-rescue:+3.3V-power") (at 87.63 50.8 0) (unit 1)
+    (in_bom yes) (on_board yes) (dnp no)
+    (property "Reference" "#PWR0104" (at 87.63 54.61 0)
+      (effects (font (size 1.27 1.27)) hide)
+    )
+    (property "Value" "+3.3V" (at 88.011 46.4058 0)
+      (effects (font (size 1.27 1.27)))
+    )
+    (property "Footprint" "" (at 87.63 50.8 0)
+      (effects (font (size 1.27 1.27)) hide)
+    )
+    (property "Datasheet" "" (at 87.63 50.8 0)
       (effects (font (size 1.27 1.27)) hide)
     )
@@
     )
   )
-  (symbol (lib_id "Device:C_Small") (at 119.38 66.04 0) (unit 1)
-    (in_bom yes) (on_board yes) (dnp no)
-    (property "Reference" "C11" (at 121.7168 64.8716 0)
+  (symbol (lib_id "Device:C_Small") (at 95.25 62.23 0) (unit 1)
+    (in_bom yes) (on_board yes) (dnp no)
+    (property "Reference" "C11" (at 97.79 60.96 0)
       (effects (font (size 1.27 1.27)) (justify left))
     )
-    (property "Value" "4.7uF" (at 114.3 68.58 0)
+    (property "Value" "4.7uF" (at 88.9 64.77 0)
       (effects (font (size 1.27 1.27)) (justify left))
     )
-    (property "Footprint" "Capacitor_SMD:C_0603_1608Metric" (at 119.38 66.04 0)
-      (effects (font (size 1.27 1.27)) hide)
-    )
-    (property "Datasheet" "~" (at 119.38 66.04 0)
+    (property "Footprint" "Capacitor_SMD:C_0603_1608Metric" (at 95.25 62.23 0)
+      (effects (font (size 1.27 1.27)) hide)
+    )
+    (property "Datasheet" "~" (at 95.25 62.23 0)
       (effects (font (size 1.27 1.27)) hide)
     )
@@
     )
   )
-  (symbol (lib_id "power:GND") (at 133.35 135.89 0) (unit 1)
-    (in_bom yes) (on_board yes) (dnp no)
-    (property "Reference" "#PWR038" (at 133.35 142.24 0)
-      (effects (font (size 1.27 1.27)) hide)
-    )
-    (property "Value" "GND" (at 133.477 140.2842 0)
-      (effects (font (size 1.27 1.27)))
-    )
-    (property "Footprint" "" (at 133.35 135.89 0)
-      (effects (font (size 1.27 1.27)) hide)
-    )
-    (property "Datasheet" "" (at 133.35 135.89 0)
+  (symbol (lib_id "power:GND") (at 78.74 64.77 0) (unit 1)
+    (in_bom yes) (on_board yes) (dnp no)
+    (property "Reference" "#PWR038" (at 78.74 71.12 0)
+      (effects (font (size 1.27 1.27)) hide)
+    )
+    (property "Value" "GND" (at 78.867 69.1642 0)
+      (effects (font (size 1.27 1.27)))
+    )
+    (property "Footprint" "" (at 78.74 64.77 0)
+      (effects (font (size 1.27 1.27)) hide)
+    )
+    (property "Datasheet" "" (at 78.74 64.77 0)
       (effects (font (size 1.27 1.27)) hide)
     )
@@
     )
   )
-  (symbol (lib_id "Device:C_Small") (at 111.76 66.04 0) (unit 1)
-    (in_bom yes) (on_board yes) (dnp no)
-    (property "Reference" "C11" (at 114.0968 64.8716 0)
+  (symbol (lib_id "Device:C_Small") (at 87.63 62.23 0) (unit 1)
+    (in_bom yes) (on_board yes) (dnp no)
+    (property "Reference" "C11" (at 89.9668 61.0616 0)
       (effects (font (size 1.27 1.27)) (justify left))
     )
-    (property "Value" "0.1uF" (at 106.68 68.58 0)
+    (property "Value" "0.1uF" (at 81.28 64.77 0)
       (effects (font (size 1.27 1.27)) (justify left))
     )
-    (property "Footprint" "Capacitor_SMD:C_0402_1005Metric" (at 111.76 66.04 0)
-      (effects (font (size 1.27 1.27)) hide)
-    )
-    (property "Datasheet" "~" (at 111.76 66.04 0)
-      (effects (font (size 1.27 1.27)) hide)
-    )
+    (property "Footprint" "Capacitor_SMD:C_0402_1005Metric" (at 87.63 62.23 0)
+      (effects (font (size 1.27 1.27)) hide)
+    )
+    (property "Datasheet" "~" (at 87.63 62.23 0)
+      (effects (font (size 1.27 1.27)) hide)
+    )
